File: Mixer Console PCB.brd (EAGLE design)
At the start: 109 parts, among them IC1 NE5532N, IC2 NE5532N, IC3 NE5532N, IC4 NE5532N, IC5 NE5532N, IC6 NE5532N, IC7 NE5532N, IC8 NE5532N, IC9 TLC339P

Commit message: WIP
Parts:
- removed C15, C19, C20: 47pf, capacitor-wima:C2.5-2
- removed C16, C17: 47u, rcl:E5-6
- removed C18: 33pf, capacitor-wima:C2.5-2
- removed C21, C23, C25, C27: 100U, rcl:E5-6
- removed C22, C24, C26, C28: 10U, rcl:E5-6
- removed D10, D11, D12, D9: (no value), SparkFun-LED:LED_3MM
- removed D3, D4, D5, D6, D7, D8: Z5.1, diode:DO34Z7
- removed IC8: NE5532N, linear:DIL08
- removed IC9: TLC339P, linear:DIL14
- removed JP1, JP2, JP3, JP4, JP5, JP6, JP7, JP8: (no value), pinhead:1X02
- removed PAD1, PAD2, PAD3, PAD4: (no value), wirepad:1,6/0,8
- removed VR1, VR2, VR3, VR4: 10k, SparkFun-Resistors:POT-PTH-ALPS
- added BASS1, EQVOL1, LINEOUT, TREB1: 100kLOG, pot:3RP/1610G
- added C29: 47nf, capacitor-wima:C2.5-2
- added C30: 560pF, capacitor-wima:C2.5-2
- added CON1, CON10, CON11, CON12, CON2, CON3, CON4, CON5, CON6, CON7, CON8, CON9: PCB-2M3, Screw Terminals:PCB2-M3
- added EQIN2, EQOUT2, FXOUT1, LINEOUT1, MIXER-OUT, MIXIN1, MIXIN2, MIXIN3, MIXIN4, MIXIN5, MIXIN6, POWERIN, POWERIN1, POWERIN2, POWERIN3, POWERIN4, POWERIN5, PREAMPOUT1, VU-IN, VU-OUT: (no value), pinhead:1X03/90
- added FADER, FXGAIN, GAIN1: 100kLOG, pot:3RP/1610N
- added J1, J5: AUDIO_JACK_TRS_0.25"_PTH_RA, SparkFun-Connectors:AUDIO_JACK_0.25"_TRS_PTH_RA
- added J2, J3: RCALOCK, SparkFun-Connectors:RCA_LOCK
- added J4: AUDIO_JACK_3.5MM_KIT, SparkFun-Connectors:AUDIO-JACK-KIT
- added LED1, LED10, LED11, LED12, LED2, LED3, LED4, LED5, LED6, LED7, LED8, LED9: (no value), led:LED3MM
- added LINE1: (no value), pot:3RP/1610G
- added R45, R46: 10k, rcl:0204/7
- added R47, R48: 4K7, rcl:0204/7
- added R49: 10K, rcl:0204/7
- added U$1, U$2: XKBENTERPRISESS-12D11G5R, XKB Enterprise SS-12D11G5R:XKBENTERPRISESS-12D11G5R
- added U$5: BOURNS 3362 100K, presetpot:POT_B64W
- C10: value 47pf -> 3N3
- C11: value 47u -> 47pf; device rcl:E5-6 -> capacitor-wima:C2.5-2
- C12: value 47u -> 47nf; device rcl:E5-6 -> capacitor-wima:C2.5-2
- C13: value 33pf -> 560pF
- C6: value 47u -> 100PF; device rcl:E5-6 -> capacitor-wima:C2.5-2
- C7: value 47u -> 100N; device rcl:E5-6 -> capacitor-wima:C2.5-2
- C8: value 33pf -> 1u
- C9: value 47pf -> 100P
- IC5: value NE5532N -> LM3915N; device linear:DIL08 -> national-semiconductor:DIL18
- R10, R28: value 1k -> 1K
- R11, R19: value 20k -> 4K7
- R12, R18, R20, R26: value 1k -> 10k
- R13, R15, R21, R23: value 4K7 -> 10k
- R16, R24, R32: value 10K -> 10k
- R17, R25: value 22k -> 10k
- R27: value 20k -> 2M2
- R29: value 4K7 -> 220k
- R30: value 10k -> 4K7
- R31: value 4K7 -> 1K
- R33: value 100klog -> 4K7; device pot:B25P -> rcl:0204/7
- R34, R35, R36: value 100klog -> 22k; device pot:B25P -> rcl:0204/7
- R37: value 330 -> 10K
- R38, R40: value 2K2 -> 22k
- R39: value 330 -> 22k
- R41: value 330 -> 10k
- R42, R44: value 2K2 -> 10k
- R43: value 330 -> 4K7
- R9: value 22k -> 1k2; device rcl:0204/7 -> rcl:0207/10
- moved C6 307.1 mm to (322.0, 50.0), turned to 0 degrees
- moved C7 292.2 mm to (322.0, 43.0), turned to 0 degrees
- moved R29 280.8 mm to (318.0, 14.0), turned to 180 degrees
- moved R10 279.5 mm to (315.0, 49.0), turned to 180 degrees
- moved R27 267.3 mm to (322.0, 47.0), turned to 180 degrees
- moved R28 261.8 mm to (322.0, 40.0), turned to 180 degrees
- moved C8 260.7 mm to (315.0, 42.0), turned to 180 degrees
- moved C9 255.5 mm to (315.0, 38.0), turned to 180 degrees
- moved R17 237.5 mm to (259.0, 18.0), turned to 0 degrees
- moved R25 234.4 mm to (258.0, 15.0), turned to 0 degrees
- moved C10 233.8 mm to (321.1, 4.30), turned to 270 degrees
- moved R31 233.7 mm to (313.0, 32.0), turned to 270 degrees
- moved IC6 232.9 mm to (318.0, 21.0), turned to 270 degrees
- moved R30 231.5 mm to (315.0, 45.0), turned to 0 degrees
- moved R13 219.8 mm to (259.0, 58.0), turned to 0 degrees
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Connections:
- removed net +12V: R33.E, R34.E, R35.E, R36.E, R37.1, R39.1, R41.1, R43.1
- removed net 0V: R33.A, R34.A, R35.A, R36.A
- removed net CLIP1: C22.-, D9.K, IC9.2
- removed net CLIP2: C24.-, D10.K, IC9.1
- removed net CLIP3: C26.-, D11.K, IC9.14
- removed net CLIP4: C28.-, D12.K, IC9.13
- removed net MIC2: C6.+, JP3.2
- removed net MIC3: C11.+, JP5.2
- removed net MIC4: C16.+, JP7.2
- removed net PREAMP2: C10.2, IC4.1, IC9.7, JP4.2, R16.1
- removed net PREAMP3: C15.2, IC6.1, IC9.9, JP6.2, R24.1
- removed net PREAMP4: C20.2, IC8.1, IC9.11, JP8.2, R32.1
- new net EQ-CH1: C14.2, IC7.1, R38.2, R41.2, R49.1
- new net EQ-CH2: C11.2, IC3.1, R34.2, R37.1, R45.2
- new net FX-BUFFER: C10.1, R31.1, U$1.LEFT
- new net FXOUT1: FXOUT1.1, FXOUT1.3, U$1.CENTER
- new net GUITARIN1: C6.2, C7.2, J5.RING, J5.TIP, R27.1, U$1.RIGHT
- new net LEFT-IN: U$2.LEFT, VU-IN.1, VU-OUT.1
- new net LEFT-MIX: IC4.2, R12.1, R13.1, R14.1, R15.1, R16.1, R17.1, R18.2
- new net LEFT1: MIXIN1.1, R12.2
- new net LEFT2: MIXIN2.1, R13.2
- new net LEFT3: MIXIN3.1, R14.2
- new net LEFT4: MIXIN4.1, R15.2
- new net LEFT5: MIXIN5.1, R16.2
- new net LEFT6: MIXIN6.1, R17.2
- new net MIX-OUT-L: IC4.1, LINEOUT.1-3, R18.1
- new net MIX-OUT-R: IC4.7, LINEOUT.2-3, R26.1
- new net N$46: BASS1.2-2, R36.1
- new net N$49: C30.2, IC3.6, R36.2
- new net N$52: C30.1, TREB1.2-2
- new net N$55: EQVOL1.2-3, IC3.7, R35.1, R46.1
- new net N$57: R46.2, TREB1.2-3
- new net N$58: R45.1, TREB1.2-1
- new net N$59: IC7.3, R48.1
- new net N$60: C14.1, IC7.2, R44.1, R49.2
- new net N$61: EQIN2.3, R44.2
- new net N$65: IC3.5, R47.1
- new net REF: IC5.8, R9.1, U$5.E
- new net RIGHT-IN: U$2.RIGHT, VU-IN.3, VU-OUT.3
- new net RIGHT-MIX: IC4.6, R20.1, R21.1, R22.1, R23.1, R24.1, R25.1, R26.2
- new net RIGHT1: MIXIN1.3, R20.2
- new net RIGHT2: MIXIN2.3, R21.2
- new net RIGHT3: MIXIN3.3, R22.2
- new net RIGHT4: MIXIN4.3, R23.2
- new net RIGHT5: MIXIN5.3, R24.2
- new net RIGHT6: MIXIN6.3, R25.2
- new net SIG: IC5.5, U$2.CENTER
- net +15V: now also IC5.3, IC5.9, LED1.A, LED10.A, LED2.A, LED3.A, LED4.A, LED5.A, LED6.A, LED7.A, LED8.A, LED9.A, POWERIN.3, POWERIN1.3, POWERIN2.3, POWERIN3.3, POWERIN4.3, POWERIN5.3, R29.1; no longer IC5.8, IC8.8, IC9.3
- net -15V: now also POWERIN.1, POWERIN1.1, POWERIN2.1, POWERIN3.1, POWERIN4.1, POWERIN5.1; no longer IC5.4, IC8.4, IC9.12
- net GND: now also C10.2, C6.1, CON1.P$1, CON1.P$2, CON10.P$1, CON10.P$2, CON11.P$1, CON11.P$2, CON12.P$1, CON12.P$2, CON2.P$1, CON2.P$2, CON3.P$1, CON3.P$2, CON4.P$1, CON4.P$2, CON5.P$1, CON5.P$2, CON6.P$1, CON6.P$2, CON7.P$1, CON7.P$2, CON8.P$1, CON8.P$2, CON9.P$1, CON9.P$2, EQIN2.2, EQOUT2.2, EQVOL1.1-1, EQVOL1.2-1, FADER.1, FXOUT1.2, IC5.2, IC5.4, J1.SLEEVE, J2.PIN, J3.PIN, J4.SLEEVE, J5.SLEEVE, LINE1.1-1, LINE1.2-1, LINEOUT.1-1, LINEOUT.2-1, LINEOUT1.2, MIXER-OUT.2, MIXIN1.2, MIXIN2.2, MIXIN3.2, MIXIN4.2, MIXIN5.2, MIXIN6.2, POWERIN.2, POWERIN1.2, POWERIN2.2, POWERIN3.2, POWERIN4.2, POWERIN5.2, PREAMPOUT1.2, R10.1, R11.2, R19.2, R27.2, R33.2, R43.2, R47.2, R48.2, U$5.A, U$5.S, VU-IN.2, VU-OUT.2; no longer C12.-, C17.-, C21.-, C23.-, C25.-, C27.-, C7.-, D3.A, D5.A, D7.A, JP1.1, JP2.1, JP3.1, JP4.1, JP5.1, JP6.1, JP7.1, JP8.1, R13.2, R15.2, R17.1, R21.2, R23.2, R25.1, R29.2, R31.2, R9.1
- net MIC1: now also J1.RING, J1.TIP; no longer JP1.2
- net N$11: now also EQOUT2.1, EQVOL1.2-2; no longer C6.-, D4.A, IC3.3, R9.2
- net N$12: now also IC3.3, R33.1; no longer C7.+, R10.2
- net N$13: now also IC4.5, R19.1; no longer C8.1, IC3.2, R10.1, R11.2
- net N$14: now also IC4.3; no longer C8.2, IC3.1, R12.2
- net N$15: now also C11.1, IC3.2, R32.1, R37.2; no longer C9.1, IC3.6, R12.1, VR2.P$3
- net N$16: now also LINE1.2-2, LINEOUT1.1; no longer IC3.5, R13.1
- net N$17: now also LINE1.1-2, LINEOUT1.3; no longer C9.2, IC3.7, R14.2, VR2.P$2
- net N$18: now also FADER.2, R6.2; no longer IC4.3, R15.1
- net N$19: now also J2.SHELL, J4.RING, LINE1.1-3; no longer C10.1, IC4.2, R14.1, R16.2
- net N$20: now also J3.SHELL, J4.TIP, LINE1.2-3; no longer D3.C, D4.C
- net N$21: now also LINEOUT.2-2, MIXER-OUT.1; no longer C11.-, D6.A, IC5.3, R17.2
- net N$22: now also LINEOUT.1-2, MIXER-OUT.3; no longer C12.+, R18.2
- net N$23: now also EQIN2.1, R32.2; no longer C13.1, IC5.2, R18.1, R19.2
- net N$24: now also IC5.6, IC5.7, R9.2; no longer C13.2, IC5.1, R19.1, R20.2
- net N$25: now also IC5.1, LED1.K; no longer C14.1, IC5.6, R20.1, VR3.P$3
- net N$26: now also IC5.18, LED2.K; no longer IC5.5, R21.1
- net N$27: now also IC5.17, LED3.K; no longer C14.2, IC5.7, R22.2, VR3.P$2
- net N$28: now also IC5.16, LED4.K; no longer IC6.3, R23.1
- net N$29: now also IC5.15, LED5.K; no longer C15.1, IC6.2, R22.1, R24.2
- net N$30: now also IC5.14, LED6.K; no longer D5.C, D6.C
- net N$31: now also IC5.13, LED7.K; no longer C16.-, D8.A, IC7.3, R25.2
- net N$32: now also IC5.12, LED8.K; no longer C17.+, R26.2
- net N$33: now also IC5.11, LED9.K; no longer C18.1, IC7.2, R26.1, R27.2
- net N$34: now also IC5.10, LED10.K; no longer C18.2, IC7.1, R27.1, R28.2
- net N$35: now also IC6.3, R28.2, R29.2; no longer C19.1, IC7.6, R28.1, VR4.P$3
- net N$36: now also BASS1.1-1, C12.2, R38.1; no longer IC7.5, R29.1
- net N$37: now also C7.1, R28.1; no longer C19.2, IC7.7, R30.2, VR4.P$2
- net N$38: now also C8.1, C9.1, IC6.2, LED11.K, LED12.A, R30.2; no longer IC8.3, R31.1
- net N$39: now also C9.2, FXGAIN.2, IC6.1, LED11.A, LED12.K, R31.2; no longer C20.1, IC8.2, R30.1, R32.2
- net N$40: now also C8.2, R10.2; no longer D7.C, D8.C
- net N$41: now also FXGAIN.1, R30.1; no longer IC9.4, PAD1.1, R33.S
- net N$42: now also BASS1.1-3, C12.1, R39.2; no longer IC9.6, PAD2.1, R34.S
- net N$43: now also BASS1.2-1, C29.2, R34.1; no longer IC9.8, PAD3.1, R35.S
- net N$44: now also BASS1.2-3, C29.1, R35.2; no longer IC9.10, PAD4.1, R36.S
- net N$45: now also BASS1.1-2, R40.1; no longer C21.+, C22.+, R37.2, R38.2
- net N$47: now also C13.2, IC7.6, R40.2; no longer D9.A, R38.1
- net N$48: now also C13.1, TREB1.1-2; no longer C23.+, C24.+, R39.2, R40.2
- net N$5: now also GAIN1.1; no longer VR1.P$3
- net N$50: now also EQVOL1.1-3, IC7.7, R39.1, R42.1; no longer D10.A, R40.1
- net N$51: now also TREB1.1-3; no longer C25.+, C26.+, R41.2
- net N$53: now also R41.1, TREB1.1-1; no longer D11.A, R42.1
- net N$54: now also IC7.5, R43.1; no longer C27.+, C28.+, R43.2, R44.2
- net N$56: now also EQOUT2.3, EQVOL1.1-2; no longer D12.A, R44.1
- net N$7: now also FADER.3, GAIN1.2; no longer R6.2, VR1.P$2
- net PREAMP1: now also PREAMPOUT1.1, PREAMPOUT1.3; no longer IC9.5, JP2.2
Routing:
- net GND: track 0.00 -> 1178.9 mm, vias 0 -> 3
- net +15V: track 0.00 -> 378.9 mm
- net -15V: track 0.00 -> 276.7 mm
- net LEFT-IN: track 0.00 -> 98.0 mm
- net REF: track 0.00 -> 96.2 mm
- net N$55: track 0.00 -> 80.3 mm, vias 0 -> 1
- net RIGHT-IN: track 0.00 -> 79.5 mm
- net LEFT-MIX: track 0.00 -> 74.4 mm
- net FX-BUFFER: track 0.00 -> 71.9 mm
- net N$50: track 0.00 -> 64.2 mm, vias 0 -> 1
- net GUITARIN1: track 0.00 -> 62.6 mm, vias 0 -> 1
- net RIGHT-MIX: track 0.00 -> 60.8 mm
- net EQ-CH1: track 0.00 -> 56.1 mm
- net N$20: track 8.86 -> 59.9 mm
- net N$24: track 11.3 -> 57.7 mm, vias 0 -> 2
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Other:
- board text added: "+ G -"
- board text added: "BAXANDALL EQ"
- board text added: "GUITAR IN"
- board text added: "INPUT"
- board text added: "L/G/R"
- board text added: "LINE-IN"
- board text added: "MIC PREAMP"
- board text added: "MIXER"
- board text added: "OUTPUT"
- board text added: "Other ideas: 555 Metronome Guitar Tuner 15-0-15v PSU (See OLD folder of this project) or TEN 3-2423 Module Headphone Amp Passthrough spare NE5532 output on OverDrv for something? FX Patching?"
- board text added: "Todo: Nothing"
- board text added: "Todo: Remove Pot Add more ports"
- board text added: "Todo: Spare Preamp Volume Control"
- board text added: "VU METER"
- board text removed: "ALL FROM https://wiredworld.tripod.com/tronics/mixer.html"

Commit message: update
Parts:
- removed EQIN2, EQOUT2, LINEOUT1, POWERIN, POWERIN1, POWERIN2, POWERIN3, POWERIN4, POWERIN5, PREAMPOUT1: (no value), pinhead:1X03/90
- added C15, C16, C17, C18, C19, C20, C21, C22, C23, C24, C25, C26: 0.1uF, capacitor-wima:C2.5-2
- added EQIN, EQOUT, LINEIN-OUT, PREAMPOUT, PWRIN, PWRIN1, PWRIN2, PWRIN3, PWRIN4, PWRIN5: Phoenix Pluggable 3.81mm 3 way, openbuilds-eagle-library:3.81MM-3WAY-PLUGGABLE-SCREW
- moved CON11 445.5 mm to (-140.0, 5.00)
- moved CON12 445.5 mm to (-140.0, 75.0), flipped to the bottom, turned to 270 degrees
- moved CON7 240.0 mm to (240.0, 75.0)
- moved CON8 240.0 mm to (240.0, 5.00)
- moved CON1 160.0 mm to (-40.0, 75.0)
- moved CON2 160.0 mm to (-40.0, 5.00), flipped to the bottom, turned to 270 degrees
- moved J1 140.0 mm to (-140.0, 63.0)
- moved C1 140.0 mm to (-126.0, 75.0)
- moved C2 140.0 mm to (-123.0, 24.5)
- moved C3 140.0 mm to (-123.0, 29.5)
- moved C4 140.0 mm to (-130.0, 44.5)
- moved C5 140.0 mm to (-123.0, 2.00)
- moved D1 140.0 mm to (-119.5, 74.0)
- moved D2 140.0 mm to (-121.5, 74.0)
- moved FADER 140.0 mm to (-136.0, 19.0)
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Connections:
- net +15V: now also C16.2, C18.2, C20.2, C22.2, C24.2, C26.2, PWRIN.3, PWRIN1.3, PWRIN2.3, PWRIN3.3, PWRIN4.3, PWRIN5.3; no longer POWERIN.3, POWERIN1.3, POWERIN2.3, POWERIN3.3, POWERIN4.3, POWERIN5.3
- net -15V: now also C15.2, C17.2, C19.2, C21.2, C23.2, C25.2, PWRIN.1, PWRIN1.1, PWRIN2.1, PWRIN3.1, PWRIN4.1, PWRIN5.1; no longer POWERIN.1, POWERIN1.1, POWERIN2.1, POWERIN3.1, POWERIN4.1, POWERIN5.1
- net GND: now also C15.1, C16.1, C17.1, C18.1, C19.1, C20.1, C21.1, C22.1, C23.1, C24.1, C25.1, C26.1, EQIN.2, EQOUT.2, LINEIN-OUT.2, PREAMPOUT.2, PWRIN.2, PWRIN1.2, PWRIN2.2, PWRIN3.2, PWRIN4.2, PWRIN5.2; no longer EQIN2.2, EQOUT2.2, LINEOUT1.2, POWERIN.2, POWERIN1.2, POWERIN2.2, POWERIN3.2, POWERIN4.2, POWERIN5.2, PREAMPOUT1.2
- net N$11: now also EQOUT.3; no longer EQOUT2.1
- net N$16: now also LINEIN-OUT.3; no longer LINEOUT1.1
- net N$17: now also LINEIN-OUT.1; no longer LINEOUT1.3
- net N$23: now also EQIN.3; no longer EQIN2.1
- net N$56: now also EQOUT.1; no longer EQOUT2.3
- net N$61: now also EQIN.1; no longer EQIN2.3
- net PREAMP1: now also PREAMPOUT.1, PREAMPOUT.3; no longer PREAMPOUT1.1, PREAMPOUT1.3
Routing:
- net GND: track 1178.9 -> 996.3 mm
- net -15V: track 276.7 -> 243.9 mm
- net PREAMP1: track 18.1 -> 31.9 mm
- net +15V: track 378.9 -> 391.8 mm, vias 0 -> 2
- net N$23: track 32.7 -> 42.8 mm
- net N$49: track 39.5 -> 49.0 mm
- net N$55: track 80.3 -> 89.8 mm
- net N$11: track 21.4 -> 30.3 mm
- net N$16: track 22.4 -> 30.9 mm
- net LEFT1: track 2.57 -> 10.6 mm
- net RIGHT1: track 4.43 -> 12.5 mm
- net N$17: track 28.5 -> 34.5 mm
- net N$50: track 64.2 -> 70.2 mm
- net N$56: track 28.8 -> 34.5 mm
- net N$47: track 34.4 -> 40.1 mm
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Other:
- board text added: "Todo: 3.81mm terminals"
- board text added: "Todo: Mic > Instrument > Line Leave effects to the Pedals"
- board text removed: "+ G -"
- board text removed: "INPUT"
- board text removed: "Todo: Spare Preamp Volume Control"
