File: Mixer Console PCB.sch (EAGLE design)
At the start: 109 parts, among them IC1 NE5532N, IC2 NE5532N, IC3 NE5532N, IC4 NE5532N, IC5 NE5532N, IC6 NE5532N, IC7 NE5532N, IC8 NE5532N, IC9 TLC339P

Commit message: WIP
Parts:
- removed C15, C19, C20: 47pf, capacitor-wima:C2.5/2
- removed C16, C17: 47u, rcl:CPOL-EUE5-6
- removed C18: 33pf, capacitor-wima:C2.5/2
- removed C21, C23, C25, C27: 100U, rcl:CPOL-EUE5-6
- removed C22, C24, C26, C28: 10U, rcl:CPOL-EUE5-6
- removed D10, D11, D12, D9: (no value), SparkFun-LED:LED3MM
- removed D3, D4, D5, D6, D7, D8: Z5.1, diode:ZENER-DIODEDO34-7
- removed IC8: NE5532N, linear:NE5532N
- removed IC9: TLC339P, linear:TLC339P
- removed JP1, JP2, JP3, JP4, JP5, JP6, JP7, JP8: (no value), pinhead:PINHD-1X2
- removed PAD1, PAD2, PAD3, PAD4: (no value), wirepad:1,6/0,8
- removed VR1, VR2, VR3, VR4: 10k, SparkFun-Resistors:POTENTIOMETER-PTH-9MM-1/20W-20%
- added BASS1, EQVOL1, LINEOUT, TREB1: 100kLOG, pot:3RP/1610G
- added C29: 47nf, capacitor-wima:C2.5/2
- added C30: 560pF, capacitor-wima:C2.5/2
- added CON1, CON10, CON11, CON12, CON2, CON3, CON4, CON5, CON6, CON7, CON8, CON9: PCB-2M3, Screw Terminals:PCB-2M3
- added EQIN2, EQOUT2, FXOUT1, LINEOUT1, MIXER-OUT, MIXIN1, MIXIN2, MIXIN3, MIXIN4, MIXIN5, MIXIN6, POWERIN, POWERIN1, POWERIN2, POWERIN3, POWERIN4, POWERIN5, PREAMPOUT1, VU-IN, VU-OUT: (no value), pinhead:PINHD-1X3/90
- added FADER, FXGAIN, GAIN1: 100kLOG, pot:3RP/1610N
- added J1, J5: AUDIO_JACK_TRS_0.25"_PTH_RA, SparkFun-Connectors:AUDIO_JACK_TRS_0.25"_PTH_RA
- added J2, J3: RCALOCK, SparkFun-Connectors:RCALOCK
- added J4: AUDIO_JACK_3.5MM_KIT, SparkFun-Connectors:AUDIO_JACK_3.5MM_KIT
- added LED1, LED10, LED11, LED12, LED2, LED3, LED4, LED5, LED6, LED7, LED8, LED9: (no value), led:LED3MM
- added LINE1: (no value), pot:3RP/1610G
- added R45, R46: 10k, rcl:R-EU_0204/7
- added R47, R48: 4K7, rcl:R-EU_0204/7
- added R49: 10K, rcl:R-EU_0204/7
- added U$1, U$2: XKBENTERPRISESS-12D11G5R, XKB Enterprise SS-12D11G5R:XKBENTERPRISESS-12D11G5R
- added U$5: BOURNS 3362 100K, presetpot:POTVERTICAL
- C10: value 47pf -> 3N3
- C11: value 47u -> 47pf; device rcl:CPOL-EUE5-6 -> capacitor-wima:C2.5/2
- C12: value 47u -> 47nf; device rcl:CPOL-EUE5-6 -> capacitor-wima:C2.5/2
- C13: value 33pf -> 560pF
- C6: value 47u -> 100PF; device rcl:CPOL-EUE5-6 -> capacitor-wima:C2.5/2
- C7: value 47u -> 100N; device rcl:CPOL-EUE5-6 -> capacitor-wima:C2.5/2
- C8: value 33pf -> 1u
- C9: value 47pf -> 100P
- IC5: value NE5532N -> LM3915N; device linear:NE5532N -> national-semiconductor:LM3915N
- R10, R28: value 1k -> 1K
- R11, R19: value 20k -> 4K7
- R12, R18, R20, R26: value 1k -> 10k
- R13, R15, R21, R23: value 4K7 -> 10k
- R16, R24, R32: value 10K -> 10k
- R17, R25: value 22k -> 10k
- R27: value 20k -> 2M2
- R29: value 4K7 -> 220k
- R30: value 10k -> 4K7
- R31: value 4K7 -> 1K
- R33: value 100klog -> 4K7; device pot:TRIM_EU-B25P -> rcl:R-EU_0204/7
- R34, R35, R36: value 100klog -> 22k; device pot:TRIM_EU-B25P -> rcl:R-EU_0204/7
- R37: value 330 -> 10K
- R38, R40: value 2K2 -> 22k
- R39: value 330 -> 22k
- R41: value 330 -> 10k
- R42, R44: value 2K2 -> 10k
- R43: value 330 -> 4K7
- R9: value 22k -> 1k2; device rcl:R-EU_0204/7 -> rcl:R-US_0207/10
Connections:
- removed net +12V: R33.E, R34.E, R35.E, R36.E, R37.1, R39.1, R41.1, R43.1
- removed net 0V: R33.A, R34.A, R35.A, R36.A
- removed net CLIP1: C22.-, D9.C, IC9A.OUT
- removed net CLIP2: C24.-, D10.C, IC9B.OUT
- removed net CLIP3: C26.-, D11.C, IC9C.OUT
- removed net CLIP4: C28.-, D12.C, IC9D.OUT
- removed net MIC2: C6.+, JP3.2
- removed net MIC3: C11.+, JP5.2
- removed net MIC4: C16.+, JP7.2
- removed net PREAMP2: C10.2, IC4A.OUT, IC9B.+IN, JP4.2, R16.1
- removed net PREAMP3: C15.2, IC6A.OUT, IC9C.+IN, JP6.2, R24.1
- removed net PREAMP4: C20.2, IC8A.OUT, IC9D.+IN, JP8.2, R32.1
- new net EQ-CH1: C14.2, IC7A.OUT, R38.2, R41.2, R49.1
- new net EQ-CH2: C11.2, IC3A.OUT, R34.2, R37.1, R45.2
- new net FX-BUFFER: C10.1, R31.1, U$1.LEFT
- new net FXOUT1: FXOUT1.1, FXOUT1.3, U$1.CENTER
- new net GUITARIN1: C6.2, C7.2, J5.RING, J5.TIP, R27.1, U$1.RIGHT
- new net LEFT-IN: U$2.LEFT, VU-IN.1, VU-OUT.1
- new net LEFT-MIX: IC4A.-IN, R12.1, R13.1, R14.1, R15.1, R16.1, R17.1, R18.2
- new net LEFT1: MIXIN1.1, R12.2
- new net LEFT2: MIXIN2.1, R13.2
- new net LEFT3: MIXIN3.1, R14.2
- new net LEFT4: MIXIN4.1, R15.2
- new net LEFT5: MIXIN5.1, R16.2
- new net LEFT6: MIXIN6.1, R17.2
- new net MIX-OUT-L: IC4A.OUT, LINEOUT/1.E, R18.1
- new net MIX-OUT-R: IC4B.OUT, LINEOUT/2.E, R26.1
- new net N$46: BASS1/2.S, R36.1
- new net N$49: C30.2, IC3B.-IN, R36.2
- new net N$52: C30.1, TREB1/2.S
- new net N$55: EQVOL1/2.E, IC3B.OUT, R35.1, R46.1
- new net N$57: R46.2, TREB1/2.E
- new net N$58: R45.1, TREB1/2.A
- new net N$59: IC7A.+IN, R48.1
- new net N$60: C14.1, IC7A.-IN, R44.1, R49.2
- new net N$61: EQIN2.3, R44.2
- new net N$65: IC3B.+IN, R47.1
- new net REF: IC5.REFADJ, R9.1, U$5.E
- new net RIGHT-IN: U$2.RIGHT, VU-IN.3, VU-OUT.3
- new net RIGHT-MIX: IC4B.-IN, R20.1, R21.1, R22.1, R23.1, R24.1, R25.1, R26.2
- new net RIGHT1: MIXIN1.3, R20.2
- new net RIGHT2: MIXIN2.3, R21.2
- new net RIGHT3: MIXIN3.3, R22.2
- new net RIGHT4: MIXIN4.3, R23.2
- new net RIGHT5: MIXIN5.3, R24.2
- new net RIGHT6: MIXIN6.3, R25.2
- new net SIG: IC5.SIGIN, U$2.CENTER
- net +15V: now also IC5.MODE, IC5.V+, LED1.A, LED10.A, LED2.A, LED3.A, LED4.A, LED5.A, LED6.A, LED7.A, LED8.A, LED9.A, POWERIN.3, POWERIN1.3, POWERIN2.3, POWERIN3.3, POWERIN4.3, POWERIN5.3, R29.1; no longer IC5P.V+, IC8P.V+, IC9P.V+
- net -15V: now also POWERIN.1, POWERIN1.1, POWERIN2.1, POWERIN3.1, POWERIN4.1, POWERIN5.1; no longer IC5P.V-, IC8P.V-, IC9P.V-
- net GND: now also C10.2, C6.1, CON1.P$1, CON1.P$2, CON10.P$1, CON10.P$2, CON11.P$1, CON11.P$2, CON12.P$1, CON12.P$2, CON2.P$1, CON2.P$2, CON3.P$1, CON3.P$2, CON4.P$1, CON4.P$2, CON5.P$1, CON5.P$2, CON6.P$1, CON6.P$2, CON7.P$1, CON7.P$2, CON8.P$1, CON8.P$2, CON9.P$1, CON9.P$2, EQIN2.2, EQOUT2.2, EQVOL1/1.A, EQVOL1/2.A, FADER.A, FXOUT1.2, IC5.RLO, IC5.V-, J1.EARTH, J2.PIN, J3.PIN, J4.SLEEVE, J5.EARTH, LINE1/1.A, LINE1/2.A, LINEOUT/1.A, LINEOUT/2.A, LINEOUT1.2, MIXER-OUT.2, MIXIN1.2, MIXIN2.2, MIXIN3.2, MIXIN4.2, MIXIN5.2, MIXIN6.2, POWERIN.2, POWERIN1.2, POWERIN2.2, POWERIN3.2, POWERIN4.2, POWERIN5.2, PREAMPOUT1.2, R10.1, R11.2, R19.2, R27.2, R33.2, R43.2, R47.2, R48.2, U$5.A, U$5.S, VU-IN.2, VU-OUT.2; no longer C12.-, C17.-, C21.-, C23.-, C25.-, C27.-, C7.-, D3.A, D5.A, D7.A, JP1.1, JP2.1, JP3.1, JP4.1, JP5.1, JP6.1, JP7.1, JP8.1, R13.2, R15.2, R17.1, R21.2, R23.2, R25.1, R29.2, R31.2, R9.1
- net MIC1: now also J1.RING, J1.TIP; no longer JP1.2
- net N$11: now also EQOUT2.1, EQVOL1/2.S; no longer C6.-, D4.A, IC3A.+IN, R9.2
- net N$12: now also IC3A.+IN, R33.1; no longer C7.+, R10.2
- net N$13: now also IC4B.+IN, R19.1; no longer C8.1, IC3A.-IN, R10.1, R11.2
- net N$14: now also IC4A.+IN; no longer C8.2, IC3A.OUT, R12.2
- net N$15: now also C11.1, IC3A.-IN, R32.1, R37.2; no longer C9.1, IC3B.-IN, R12.1, VR2.A
- net N$16: now also LINE1/2.S, LINEOUT1.1; no longer IC3B.+IN, R13.1
- net N$17: now also LINE1/1.S, LINEOUT1.3; no longer C9.2, IC3B.OUT, R14.2, VR2.S
- net N$18: now also FADER.S, R6.2; no longer IC4A.+IN, R15.1
- net N$19: now also J2.SHELL, J4.RING, LINE1/1.E; no longer C10.1, IC4A.-IN, R14.1, R16.2
- net N$20: now also J3.SHELL, J4.TIP, LINE1/2.E; no longer D3.C, D4.C
- net N$21: now also LINEOUT/2.S, MIXER-OUT.1; no longer C11.-, D6.A, IC5A.+IN, R17.2
- net N$22: now also LINEOUT/1.S, MIXER-OUT.3; no longer C12.+, R18.2
- net N$23: now also EQIN2.1, R32.2; no longer C13.1, IC5A.-IN, R18.1, R19.2
- net N$24: now also IC5.REFOUT, IC5.RHI, R9.2; no longer C13.2, IC5A.OUT, R19.1, R20.2
- net N$25: now also IC5.LED1, LED1.C; no longer C14.1, IC5B.-IN, R20.1, VR3.A
- net N$26: now also IC5.LED2, LED2.C; no longer IC5B.+IN, R21.1
- net N$27: now also IC5.LED3, LED3.C; no longer C14.2, IC5B.OUT, R22.2, VR3.S
- net N$28: now also IC5.LED4, LED4.C; no longer IC6A.+IN, R23.1
- net N$29: now also IC5.LED5, LED5.C; no longer C15.1, IC6A.-IN, R22.1, R24.2
- net N$30: now also IC5.LED6, LED6.C; no longer D5.C, D6.C
- net N$31: now also IC5.LED7, LED7.C; no longer C16.-, D8.A, IC7A.+IN, R25.2
- net N$32: now also IC5.LED8, LED8.C; no longer C17.+, R26.2
- net N$33: now also IC5.LED9, LED9.C; no longer C18.1, IC7A.-IN, R26.1, R27.2
- net N$34: now also IC5.LED10, LED10.C; no longer C18.2, IC7A.OUT, R27.1, R28.2
- net N$35: now also IC6A.+IN, R28.2, R29.2; no longer C19.1, IC7B.-IN, R28.1, VR4.A
- net N$36: now also BASS1/1.A, C12.2, R38.1; no longer IC7B.+IN, R29.1
- net N$37: now also C7.1, R28.1; no longer C19.2, IC7B.OUT, R30.2, VR4.S
- net N$38: now also C8.1, C9.1, IC6A.-IN, LED11.C, LED12.A, R30.2; no longer IC8A.+IN, R31.1
- net N$39: now also C9.2, FXGAIN.S, IC6A.OUT, LED11.A, LED12.C, R31.2; no longer C20.1, IC8A.-IN, R30.1, R32.2
- net N$40: now also C8.2, R10.2; no longer D7.C, D8.C
- net N$41: now also FXGAIN.A, R30.1; no longer IC9A.-IN, PAD1.P, R33.S
- net N$42: now also BASS1/1.E, C12.1, R39.2; no longer IC9B.-IN, PAD2.P, R34.S
- net N$43: now also BASS1/2.A, C29.2, R34.1; no longer IC9C.-IN, PAD3.P, R35.S
- net N$44: now also BASS1/2.E, C29.1, R35.2; no longer IC9D.-IN, PAD4.P, R36.S
- net N$45: now also BASS1/1.S, R40.1; no longer C21.+, C22.+, R37.2, R38.2
- net N$47: now also C13.2, IC7B.-IN, R40.2; no longer D9.A, R38.1
- net N$48: now also C13.1, TREB1/1.S; no longer C23.+, C24.+, R39.2, R40.2
- net N$5: now also GAIN1.A; no longer VR1.A
- net N$50: now also EQVOL1/1.E, IC7B.OUT, R39.1, R42.1; no longer D10.A, R40.1
- net N$51: now also TREB1/1.E; no longer C25.+, C26.+, R41.2
- net N$53: now also R41.1, TREB1/1.A; no longer D11.A, R42.1
- net N$54: now also IC7B.+IN, R43.1; no longer C27.+, C28.+, R43.2, R44.2
- net N$56: now also EQOUT2.3, EQVOL1/1.S; no longer D12.A, R44.1
- net N$7: now also FADER.E, GAIN1.S; no longer R6.2, VR1.S
- net PREAMP1: now also PREAMPOUT1.1, PREAMPOUT1.3; no longer IC9A.+IN, JP2.2
Other:
- note added: "FROM https://wiredworld.tripod.com/tronics/mixer.html"
- note added: "From https://sound-au.com/dwopa2.htm#s7"
- note added: "Mounting"
- note added: "Power Input"
- note added: "Stage 0: Input and Transient Protection"
- note added: "Stage 1: Inverting, Unity Gain Low Impedance drive for EQ"
- note added: "Stage 1: Non Inverting, 26dB Fixed Gain"
- note added: "Stage 2: Baxandall Equalizer"
- note added: "Stage 2: Inverting, Variable Gain"
- note added: "Stage 3: Inverting (correcting stage 2), Unity Gain"
- note added: "Stage 3: Inverting, Unity Gain"
- note added: "This circuit must be driven from a low impedance, so connecting it after the volume control (for example) is a no-no. Ideally, the output of an opamp will be the source, thus ensuring the required low impedance."
- note added: "https://guitarpcb.com/wp-content/uploads/2018/06/BD_Shredding-Eagle.pdf"
- note removed: "ADJUST TO 2V"

Commit message: update
Parts:
- removed EQIN2, EQOUT2, LINEOUT1, POWERIN, POWERIN1, POWERIN2, POWERIN3, POWERIN4, POWERIN5, PREAMPOUT1: (no value), pinhead:PINHD-1X3/90
- added C15, C16, C17, C18, C19, C20, C21, C22, C23, C24, C25, C26: 0.1uF, capacitor-wima:C2.5/2
- added EQIN, EQOUT, LINEIN-OUT, PREAMPOUT, PWRIN, PWRIN1, PWRIN2, PWRIN3, PWRIN4, PWRIN5: Phoenix Pluggable 3.81mm 3 way, openbuilds-eagle-library:CONNECTOR-M3
Connections:
- net +15V: now also C16.2, C18.2, C20.2, C22.2, C24.2, C26.2, PWRIN.3, PWRIN1.3, PWRIN2.3, PWRIN3.3, PWRIN4.3, PWRIN5.3; no longer POWERIN.3, POWERIN1.3, POWERIN2.3, POWERIN3.3, POWERIN4.3, POWERIN5.3
- net -15V: now also C15.2, C17.2, C19.2, C21.2, C23.2, C25.2, PWRIN.1, PWRIN1.1, PWRIN2.1, PWRIN3.1, PWRIN4.1, PWRIN5.1; no longer POWERIN.1, POWERIN1.1, POWERIN2.1, POWERIN3.1, POWERIN4.1, POWERIN5.1
- net GND: now also C15.1, C16.1, C17.1, C18.1, C19.1, C20.1, C21.1, C22.1, C23.1, C24.1, C25.1, C26.1, EQIN.2, EQOUT.2, LINEIN-OUT.2, PREAMPOUT.2, PWRIN.2, PWRIN1.2, PWRIN2.2, PWRIN3.2, PWRIN4.2, PWRIN5.2; no longer EQIN2.2, EQOUT2.2, LINEOUT1.2, POWERIN.2, POWERIN1.2, POWERIN2.2, POWERIN3.2, POWERIN4.2, POWERIN5.2, PREAMPOUT1.2
- net N$11: now also EQOUT.3; no longer EQOUT2.1
- net N$16: now also LINEIN-OUT.3; no longer LINEOUT1.1
- net N$17: now also LINEIN-OUT.1; no longer LINEOUT1.3
- net N$23: now also EQIN.3; no longer EQIN2.1
- net N$56: now also EQOUT.1; no longer EQOUT2.3
- net N$61: now also EQIN.1; no longer EQIN2.3
- net PREAMP1: now also PREAMPOUT.1, PREAMPOUT.3; no longer PREAMPOUT1.1, PREAMPOUT1.3
